Commit message: Modify the tablebot URDF to represent the automatic calibration setup (caltab connected to the EE)

File: urdf/ur5_table.urdf.xacro (robot description, xacro)
@@ -3,9 +3,4 @@
   <xacro:include filename="$(find ur_description)/urdf/common.gazebo.xacro" />
   <xacro:include filename="$(find ur_description)/urdf/ur5.urdf.xacro" />
-  <xacro:include filename="$(find iai_kms_40_description)/urdf/kms_40.urdf.xacro"/>
-  <xacro:include filename="$(find iai_adapters_description)/urdf/adapter_fwa050_wsg50.urdf.xacro"/>
-  <xacro:include filename="$(find iai_adapters_description)/urdf/adapter_kms40_fwk050.urdf.xacro"/>
-  <xacro:include filename="$(find iai_adapters_description)/urdf/fwk_fwa_050.urdf.xacro"/>
-  <xacro:include filename="$(find iai_wsg_50_description)/urdf/wsg_50.urdf.xacro"/>
   <material name="gray">
     <color rgba="0.56 0.67 0.67 1"/>
@@ -59,32 +54,23 @@
       <origin xyz="0.0 0.0 ${arm_mounting_plate_height}" rpy="0 0 -${pi/4}" />
     </joint>
-    <link name="kms_mounting_plate">
+    <link name="caltab_link">
       <visual>
         <geometry>
-          <mesh filename="package://iai_table_robot_description/meshes/adapter_plate_iso50_kms40_weiss.stl" scale="0.001 0.001 0.001"/>
+          <mesh filename="package://iai_table_robot_description/meshes/caltab_complete.stl"/>
         </geometry>
         <material name="gray"/>
       </visual>
+      <collision>
+        <geometry>
+          <mesh filename="package://iai_table_robot_description/meshes/caltab_complete.stl"/>
+        </geometry>
+        <material name="gray"/>
+      </collision>
     </link>
-    <joint name="kms_mounting_plate_joint" type="fixed">
-      <parent link="ee_link" />
-      <child link="kms_mounting_plate" />
-      <origin xyz="0 0 0" rpy="0 ${pi/2} 0" />
+    <joint name="caltab_link" type="fixed">
+      <parent link="tool0" />
+      <child link="caltab_link" />
+      <origin xyz="0.0 0.0 0.0" rpy="0 0 -${pi/2}" />
     </joint>
-    <kms_40_xacro parent="kms_mounting_plate" prefix="">
-      <origin xyz="0 0 0" rpy="0 0 0" />
-    </kms_40_xacro>
-    <adapter_kms40_fwk050_xacro parent="kms40_frame_out" prefix="">
-      <origin xyz="0 0 0" rpy="0 0 0" />
-    </adapter_kms40_fwk050_xacro>
-    <fwk_fwa_050_xacro parent="adapter_kms40_fwk050_frame_out" prefix="">
-      <origin xyz="0 0 0" rpy="0 0 0" />
-    </fwk_fwa_050_xacro>
-    <adapter_fwa050_wsg50_xacro parent="fwk_fwa_050_frame_out" prefix="">
-      <origin xyz="0 0 0.0" rpy="0 0 0" />
-    </adapter_fwa050_wsg50_xacro>
-    <wsg_50_xacro name="gripper" parent="adapter_fwa050_wsg50_frame_out">
-      <origin xyz="0 0 0" rpy="0 0 3.14159265359"/>
-    </wsg_50_xacro>
   </xacro:macro>
 </robot>
